Commit message: removed EE urdf

File: src/manipulation/lbr_description/urdf/med7/med7_description.xacro (robot description, xacro)
@@ -266,39 +266,10 @@
             </collision>
         </link>
-  	<!-- Joint connecting Link 7 to End Effector -->
         <joint name="${robot_name}_joint_ee" type="fixed">
             <parent link="${robot_name}_link_7" />
             <child link="${robot_name}_link_ee" />
-            <origin xyz="-0.046 0 0.161" rpy="0 0 0" />
-        </joint>
-        <!-- End Effector (Link EE) -->
+            <origin xyz="0 0 0.035" rpy="0 0 0" />
+        </joint>
         <link name="${robot_name}_link_ee">
-            <!-- Inertial properties -->
-            <inertial>
-                <origin rpy="0 0 0" xyz="0.0 -0.029824 0.076267" />
-                <mass value="1.474048" />
-                <inertia ixx="0.008179" ixy="0.0" ixz="0.0"
-                        iyy="0.006879" iyz="0.002704"
-                        izz="0.003709"/>
-            </inertial>
-            <!-- Visual representation -->
-            <visual>
-                <origin rpy="3.1415926 0 3.1415926" xyz="0 0 0"/>
-                <geometry>
-                    <mesh filename="package://lbr_description/meshes/med7/visual/end_effector_worx_with_d405.stl"
-                          scale="0.001 0.001 0.001"/>
-                </geometry>
-                <material name="blue">
-                    <color rgba=".5 .9 1 1"/>
-                </material>
-            </visual>
-            <!-- Collision geometry -->
-            <collision>
-                <origin rpy="3.1415926 0 3.1415926" xyz="0 0 0"/>
-                <geometry>
-                    <mesh filename="package://lbr_description/meshes/med7/collision/end_effector_worx_with_d405.stl"
-                          scale="0.001 0.001 0.001"/>
-                </geometry>
-            </collision>
         </link>
     </xacro:macro>

Commit message: Added effector urdf

File: src/manipulation/lbr_description/urdf/med7/med7_description.xacro (robot description, xacro)
@@ -272,4 +272,25 @@
         </joint>
         <link name="${robot_name}_link_ee">
+            <inertial>
+            <!-- The CoM is 15.4 cm below the link's origin, along Z. There is no rotation of the inertial frame -->
+                <origin rpy="0 0 0" xyz="0.0 0.0 -0.154" />
+                <mass value="0.674" />
+                <inertia ixx="0.008179" ixy="0.0" ixz="0.0" iyy="0.006879" iyz="0.002704" izz="0.003709" />
+            </inertial>
+            <visual>
+                <origin rpy="0 3.14157 0.0" xyz="0.0 0.0 0.154" />
+                <geometry>
+                    <mesh filename="package://lbr_description/meshes/med7/visual/worx+motor+mount+refined+3.stl" scale="0.001 0.001 0.001" />
+                </geometry>
+                <material name="blue">
+                    <color rgba="0.5 0.9 1 1.0" />
+                </material>
+            </visual>
+            <collision>
+                <origin rpy="0 3.14157 0" xyz="0.0 0.0 0.1694" />
+                <geometry>
+                    <mesh filename="package://lbr_description/meshes/med7/collision/worx+motor+mount+refined+3.stl" scale="0.0011 0.0011 0.0011" />
+                </geometry>
+            </collision>
         </link>
     </xacro:macro>

Commit message: Corrected EE Frame

File: src/manipulation/lbr_description/urdf/med7/med7_description.xacro (robot description, xacro)
@@ -269,15 +269,15 @@
             <parent link="${robot_name}_link_7" />
             <child link="${robot_name}_link_ee" />
-            <origin xyz="0 0 0.035" rpy="0 0 0" />
+            <!-- <origin xyz="0 0 0.035" rpy="0 0 0" /> -->
+            <origin xyz="0 0 0.189" rpy="0 0 0" />
         </joint>
         <link name="${robot_name}_link_ee">
             <inertial>
-            <!-- The CoM is 15.4 cm below the link's origin, along Z. There is no rotation of the inertial frame -->
-                <origin rpy="0 0 0" xyz="0.0 0.0 -0.154" />
+                <origin rpy="0 0 0" xyz="0.0 0.0 0.0" />
                 <mass value="0.674" />
                 <inertia ixx="0.008179" ixy="0.0" ixz="0.0" iyy="0.006879" iyz="0.002704" izz="0.003709" />
             </inertial>
             <visual>
-                <origin rpy="0 3.14157 0.0" xyz="0.0 0.0 0.154" />
+                <origin rpy="0 3.14157 0.0" xyz="0.0 0.0 0.0" />
                 <geometry>
                     <mesh filename="package://lbr_description/meshes/med7/visual/worx+motor+mount+refined+3.stl" scale="0.001 0.001 0.001" />
@@ -288,5 +288,5 @@
             </visual>
             <collision>
-                <origin rpy="0 3.14157 0" xyz="0.0 0.0 0.1694" />
+                <origin rpy="0 3.14157 0" xyz="0.0 0.0 0.0" />
                 <geometry>
                     <mesh filename="package://lbr_description/meshes/med7/collision/worx+motor+mount+refined+3.stl" scale="0.0011 0.0011 0.0011" />
